Commit message: HW2:Fixes in robot description, added navigation

File: ya_rover_description/urdf/components/base/base.urdf.xacro (robot description, xacro)
@@ -10,13 +10,13 @@
         <geometry>
           <!-- <box size="1.2 0.6 0.5"/> -->
-          <mesh filename="file://$(find ya_rover_description)/meshes/wheels/base_orig.dae" scale="1.0 1.0 1.0"/>
+          <mesh filename="file://$(find ya_rover_description)/meshes/wheels/base_orig.dae" scale="0.5 0.5 0.5"/>
         </geometry>
-        <origin xyz="0.0 -0.07 -0.5" rpy="0 0 0"/>
+        <origin xyz="0.0 -0.07 -0.5" rpy="0 0 ${pi/2}"/>
       </visual>
       <collision>
         <geometry>
-          <box size="0.9 1.7 1.0"/>
+          <box size="0.68 0.95 0.365"/>
         </geometry>
-        <origin xyz="0 0 0" rpy="0 0 0"/>
+        <origin xyz="-0.03 -0.06 -0.12" rpy="0 0 ${pi/2}"/>
       </collision>
       <inertial>

File: ya_rover_description/urdf/components/sensors/lidar.urdf.xacro (robot description, xacro)
@@ -13,13 +13,13 @@
     <link name="${prefix}_link">
       <visual>
-        <origin xyz="0.0 0.0 0.0" rpy="0 0 0"/>
+        <origin xyz="0.0 0.0 0.0" rpy="0 0 ${pi/2}"/>
         <geometry>
-            <mesh filename="file://$(find ya_rover_description)/meshes/sensors/lidar_flag.dae" scale="0.5 0.5 0.5"/>
+            <mesh filename="file://$(find ya_rover_description)/meshes/sensors/lidar_flag.dae" scale="0.25 0.25 0.25"/>
         </geometry>
       </visual>
       <collision>
-			<origin xyz="0.0 -0.0 0.0" rpy="0 0 0"/>
+			<origin xyz="-0.11 -0.0 -0.43" rpy="0 0 ${pi/2}"/>
 			<geometry>
-				<mesh filename="file://$(find ya_rover_description)/meshes/sensors/lidar.stl" scale="0.5 0.5 0.5"/>
+				<mesh filename="file://$(find ya_rover_description)/meshes/sensors/lidar.stl" scale="0.25 0.25 0.25"/>
 			</geometry>
       <material name="color_black"/>

File: ya_rover_description/urdf/components/wheels/wheel.urdf.xacro (robot description, xacro)
@@ -6,12 +6,14 @@
   <xacro:macro name="wheel_macro" params="prefix parent name xyz rpy side">
     <xacro:if value="${side == 'left'}">
-    <xacro:property name="wheel_rpy_visual" value="0 0 0"/>
+    <xacro:property name="wheel_rpy_visual" value="0 0 ${pi/2}"/>
     <xacro:property name="wheel_xyz_visual" value="0.0 0.0 0.0"/>
-    <xacro:property name="offset" value="0.1 0 0"/>
+    <xacro:property name="offset" value="0.0 0 0"/>
+    <xacro:property name="axx" value=" 0 1 0"/>
     </xacro:if>
     <xacro:if value="${side == 'right'}">
-    <xacro:property name="wheel_rpy_visual" value="0 0 0"/>
+    <xacro:property name="wheel_rpy_visual" value="0 0 ${pi/2}"/>
     <xacro:property name="wheel_xyz_visual" value="0 0 0"/>
-    <xacro:property name="offset" value="-0.1 0 0"/>
+    <xacro:property name="offset" value="-0.0 0 0"/>
+    <xacro:property name="axx" value=" 0 -1 0"/>
     </xacro:if>
     <xacro:property name="wheel_radius" value="0.1"/>
@@ -22,5 +24,5 @@
       <visual>
         <geometry>
-          <mesh filename="file://$(find ya_rover_description)/meshes/wheels/wheel_final.stl" scale="1.0 1.0 1.0"/>
+          <mesh filename="file://$(find ya_rover_description)/meshes/wheels/wheel_final.stl" scale="0.5 0.5 0.5"/>
           <!-- <cylinder length="0.11" radius="0.15"/> -->
         </geometry>
@@ -33,7 +35,7 @@
         <geometry>
         <!-- <mesh filename="file://$(find ya_rover_description)/meshes/wheels/wheel2.stl" scale="1.2 1.2 1.2"/> -->
-          <cylinder length="0.13" radius="0.24"/>
+          <cylinder length="0.065" radius="0.12"/>
         </geometry>
-        <origin xyz="${offset}" rpy="0 ${pi/2} 0"/>
+        <origin xyz="${offset}" rpy="0 ${pi/2} ${pi/2}"/>
         <material name="color_black"/>
       </collision>
@@ -48,5 +50,5 @@
       <child link="${prefix}${name}"/>
       <origin xyz="${xyz}" rpy="${rpy}"/>
-      <axis xyz="1 0 0"/>
+      <axis xyz="${axx}"/>
       <limit effort="10" velocity="10" lower="-1000" upper="1000"/>
       <mass value="${wheel_mass}"/>

File: ya_rover_description/urdf/robots/ya_rover.urdf.xacro (robot description, xacro)
@@ -10,12 +10,12 @@
     <xacro:include filename="$(find ya_rover_description)/urdf/components/plugins/transmission.urdf.xacro" />
     <xacro:base/>
-    <xacro:wheel_macro prefix="" parent="base_link" name="wheel_front_left" xyz="0.55 -0.6 -0.43" rpy="0 0 0" side="left"/>
-    <xacro:wheel_macro prefix="" parent="base_link" name="wheel_front_right" xyz="-0.55001 -0.6 -0.43" rpy="0 0 0" side="right"/>
-    <xacro:wheel_macro prefix="" parent="base_link" name="wheel_middle_left" xyz="0.55 0.053 -0.43" rpy="0 0 0" side="left"/>
-    <xacro:wheel_macro prefix="" parent="base_link" name="wheel_middle_right" xyz="-0.55001 0.053 -0.43" rpy="0 0 0" side="right"/>
-    <xacro:wheel_macro prefix="" parent="base_link" name="wheel_rear_left" xyz="0.55 0.733 -0.43" rpy="0 0 0" side="left"/>
-    <xacro:wheel_macro prefix="" parent="base_link" name="wheel_rear_right" xyz="-0.55001 0.733 -0.43" rpy="0 0 0" side="right"/>
+    <xacro:wheel_macro prefix="" parent="base_link" name="wheel_front_left" xyz="0.26 0.23 -0.47" rpy="0 0 0" side="left"/>
+    <xacro:wheel_macro prefix="" parent="base_link" name="wheel_front_right" xyz="0.26 -0.35 -0.47" rpy="0 0 ${-pi}" side="right"/>
+    <xacro:wheel_macro prefix="" parent="base_link" name="wheel_middle_left" xyz="-0.06 0.23 -0.47" rpy="0 0 0" side="left"/>
+    <xacro:wheel_macro prefix="" parent="base_link" name="wheel_middle_right" xyz="-0.06 -0.35 -0.47" rpy="0 0 ${-pi}" side="right"/>
+    <xacro:wheel_macro prefix="" parent="base_link" name="wheel_rear_left" xyz="-0.40 0.23 -0.47" rpy="0 0 0" side="left"/>
+    <xacro:wheel_macro prefix="" parent="base_link" name="wheel_rear_right" xyz="-0.40 -0.35 -0.47" rpy="0 0 ${-pi}" side="right"/>
     <xacro:lidar prefix="lidar" parent="base_link">
-        <origin xyz="0.0 -0.61 0.81" rpy="0.0 0.0 0.0"/>
+        <origin xyz="0.29 -0.05 0.13" rpy="0.0 0.0 0.0"/>
     </xacro:lidar>
     <xacro:control>
