Commit message: add navigation and split into folders

File: f1_description/urdf/f1.urdf.xacro (robot description, xacro)
@@ -1,4 +1,4 @@
 <?xml version="1.0"?>
-<robot name="charli" xmlns:xacro="http://ros.org/wiki/xacro">
+<robot name="f1" xmlns:xacro="http://ros.org/wiki/xacro">
   <material name="Black">
     <color rgba="0 0 0 1" />
@@ -13,11 +13,10 @@
     <color rgba="1 1 1 1" />
   </material>
-  <link name="base_link" />
-  <!-- Chassis -->
-  <link name="chassis">
+  <link name="base_footprint"/>
+  <link name="base_link">
     <collision>
       <origin xyz="0 0 0" rpy="0 0 1.57" />
       <geometry>
-				<mesh filename="file://$(find charli)/urdf/meshes/chassis.dae" scale="0.3 0.3 0.3"/>
+				<mesh filename="file://$(find f1_description)/urdf/meshes/chassis.dae" scale="0.3 0.3 0.3"/>
       </geometry>
     </collision>
@@ -25,5 +24,5 @@
       <origin xyz="0 0 0" rpy="0 0 1.57" />
       <geometry>
-				<mesh filename="file://$(find charli)/urdf/meshes/chassis.dae" scale="0.3 0.3 0.3"/>
+				<mesh filename="file://$(find f1_description)/urdf/meshes/chassis.dae" scale="0.3 0.3 0.3"/>
       </geometry>
       <!-- <material name="Orange" /> -->
@@ -35,8 +34,8 @@
     </inertial>
   </link>
-  <joint name="chassis_joint" type="fixed">
-    <origin xyz="0.8 0 0.5" rpy="0 0 0" />
-    <parent link="base_link" />
-    <child link="chassis" />
+  <joint name="base_footprint_joint" type="fixed">
+    <parent link="base_footprint"/>
+    <child link="base_link"/>
+    <origin xyz="0 0 0.5" rpy="0 0 0"/>
   </joint>
   <!-- rear left wheel Link -->
@@ -44,14 +43,14 @@
     <collision>
       <geometry>
-				<mesh filename="file://$(find charli)/urdf/meshes/wheel_collision.dae" scale="0.3 0.3 0.3"/>
-      </geometry>
-    </collision>
-    <visual>
-      <geometry>
-				<mesh filename="file://$(find charli)/urdf/meshes/wheel.dae" scale="0.3 0.3 0.3"/>
-      </geometry>
-    </visual>
-    <inertial>
-      <mass value="11.3" />
+				<mesh filename="file://$(find f1_description)/urdf/meshes/wheel_collision.dae" scale="0.3 0.3 0.3"/>
+      </geometry>
+    </collision>
+    <visual>
+      <geometry>
+				<mesh filename="file://$(find f1_description)/urdf/meshes/wheel.dae" scale="0.3 0.3 0.3"/>
+      </geometry>
+    </visual>
+    <inertial>
+      <mass value="1.3" />
       <inertia ixx="0.26" ixy="0.0" ixz="0.0" iyy="0.26" iyz="0.0" izz="0.51" />
     </inertial>
@@ -59,8 +58,8 @@
   <joint name="rear_left_wheel_joint" type="continuous">
     <origin xyz="-0.8 0.65 -0.1" rpy="-1.57 0 0" />
-    <parent link="chassis" />
+    <parent link="base_link" />
     <child link="rear_left_wheel" />
     <axis xyz="0 0 1" />
-    <dynamics damping="0.2" />
+    <dynamics damping="0" />
   </joint>
   <!-- rear right wheel Link -->
@@ -68,14 +67,14 @@
     <collision>
       <geometry>
-				<mesh filename="file://$(find charli)/urdf/meshes/wheel_collision.dae" scale="0.3 0.3 0.3"/>
-      </geometry>
-    </collision>
-    <visual>
-      <geometry>
-				<mesh filename="file://$(find charli)/urdf/meshes/wheel_1.dae" scale="0.3 0.3 0.3"/>
-      </geometry>
-    </visual>
-    <inertial>
-      <mass value="11.3" />
+				<mesh filename="file://$(find f1_description)/urdf/meshes/wheel_collision.dae" scale="0.3 0.3 0.3"/>
+      </geometry>
+    </collision>
+    <visual>
+      <geometry>
+				<mesh filename="file://$(find f1_description)/urdf/meshes/wheel_1.dae" scale="0.3 0.3 0.3"/>
+      </geometry>
+    </visual>
+    <inertial>
+      <mass value="1.3" />
       <inertia ixx="0.26" ixy="0.0" ixz="0.0" iyy="0.26" iyz="0.0" izz="0.51" />
     </inertial>
@@ -83,8 +82,8 @@
   <joint name="rear_right_wheel_joint" type="continuous">
     <origin xyz="-0.8 -0.65 -0.1" rpy="-1.57 0 0" />
-    <parent link="chassis" />
+    <parent link="base_link" />
     <child link="rear_right_wheel" />
     <axis xyz="0 0 1" />
-    <dynamics damping="0.2" />
+    <dynamics damping="0" />
   </joint>
   <!-- left steer Link -->
@@ -97,8 +96,8 @@
   <joint name="left_wheel_steering_joint" type="revolute">
     <origin xyz="1.37 0.65 -0.1" rpy="0 0 0" />
-    <parent link="chassis" />
+    <parent link="base_link" />
     <child link="left_wheel_steering" />
     <axis xyz="0 0 1" />
-    <dynamics damping="0.2" />
+    <dynamics damping="0" />
     <limit effort="1000.0" lower="-0.523599" upper="0.523599" velocity="30"/>
   </joint>
@@ -112,8 +111,8 @@
   <joint name="right_wheel_steering_joint" type="revolute">
     <origin xyz="1.37 -0.65 -0.1" rpy="0 0 0" />
-    <parent link="chassis" />
+    <parent link="base_link" />
     <child link="right_wheel_steering" />
     <axis xyz="0 0 1" />
-    <dynamics damping="0.2" />
+    <dynamics damping="0" />
     <limit effort="1000.0" lower="-0.523599" upper="0.523599" velocity="30"/>
   </joint>
@@ -122,14 +121,14 @@
     <collision>
       <geometry>
-				<mesh filename="file://$(find charli)/urdf/meshes/wheel_collision.dae" scale="0.3 0.3 0.3"/>
-      </geometry>
-    </collision>
-    <visual>
-      <geometry>
-				<mesh filename="file://$(find charli)/urdf/meshes/wheel.dae" scale="0.3 0.3 0.3"/>
-      </geometry>
-    </visual>
-    <inertial>
-      <mass value="11.3" />
+				<mesh filename="file://$(find f1_description)/urdf/meshes/wheel_collision.dae" scale="0.3 0.3 0.3"/>
+      </geometry>
+    </collision>
+    <visual>
+      <geometry>
+				<mesh filename="file://$(find f1_description)/urdf/meshes/wheel.dae" scale="0.3 0.3 0.3"/>
+      </geometry>
+    </visual>
+    <inertial>
+      <mass value="1.3" />
       <inertia ixx="0.26" ixy="0.0" ixz="0.0" iyy="0.26" iyz="0.0" izz="0.51" />
     </inertial>
@@ -140,5 +139,5 @@
     <child link="front_left_wheel" />
     <axis xyz="0 0 1" />
-    <dynamics damping="0.2" />
+    <dynamics damping="0" />
   </joint>
   <!-- front right wheel Link -->
@@ -146,14 +145,14 @@
     <collision>
       <geometry>
-				<mesh filename="file://$(find charli)/urdf/meshes/wheel_collision.dae" scale="0.3 0.3 0.3"/>
-      </geometry>
-    </collision>
-    <visual>
-      <geometry>
-				<mesh filename="file://$(find charli)/urdf/meshes/wheel_1.dae" scale="0.3 0.3 0.3"/>
-      </geometry>
-    </visual>
-    <inertial>
-      <mass value="11.3" />
+				<mesh filename="file://$(find f1_description)/urdf/meshes/wheel_collision.dae" scale="0.3 0.3 0.3"/>
+      </geometry>
+    </collision>
+    <visual>
+      <geometry>
+				<mesh filename="file://$(find f1_description)/urdf/meshes/wheel_1.dae" scale="0.3 0.3 0.3"/>
+      </geometry>
+    </visual>
+    <inertial>
+      <mass value="1.3" />
       <inertia ixx="0.26" ixy="0.0" ixz="0.0" iyy="0.26" iyz="0.0" izz="0.51" />
     </inertial>
@@ -164,10 +163,10 @@
     <child link="front_right_wheel" />
     <axis xyz="0 0 1" />
-    <dynamics damping="0.2" />
+    <dynamics damping="0" />
   </joint>
   <joint name="lidar_joint" type="fixed">
     <parent link="base_link"/>
     <child link="lidar_link"/>
-    <origin xyz="2.8 0 0.5" rpy="0 0 0" />
+    <origin xyz="1.8 0 0.5" rpy="0 0 0" />
   </joint>
     <link name="lidar_link">
@@ -175,5 +174,5 @@
         <origin xyz="0 0 0" rpy="0 0 0"/>
         <geometry>
-            <mesh filename="file://$(find charli)/urdf/meshes/hokuyo_urg_04lx_ug01.stl"/>
+            <mesh filename="file://$(find f1_description)/urdf/meshes/hokuyo_urg_04lx_ug01.stl"/>
         </geometry>
       </visual>
@@ -181,5 +180,5 @@
 			<origin xyz="0 0 0" rpy="0 0 0"/>
 			<geometry>
-				<mesh filename="file://$(find charli)/urdf/meshes/hokuyo_urg_04lx_ug01.stl"/>
+				<mesh filename="file://$(find f1_description)/urdf/meshes/hokuyo_urg_04lx_ug01.stl"/>
 			</geometry>
 	  </collision>
@@ -223,7 +222,25 @@
     </joint>
   </ros2_control>
-  <gazebo>
+  <!-- <gazebo>
     <plugin filename="gz_ros2_control-system" name="gz_ros2_control::GazeboSimROS2ControlPlugin">
-      <parameters>$(find charli)/config/ackermann_drive_controller.yaml</parameters>
+      <parameters>$(find f1_control)/config/ackermann_drive_controller.yaml</parameters>
+      	<ros>
+					<namespace>f1</namespace>
+					<remapping>tf:=/f1/tf</remapping>
+					<remapping>tf_static:=/f1/tf_static</remapping>
+					<remapping>ackermann_steering_controller/odometry:=odom</remapping>
+          			<remapping>ackermann_steering_controller/tf_odometry:=tf</remapping>
+				</ros>
+    </plugin>
+  </gazebo> -->
+    <gazebo>
+    <plugin filename="gz_ros2_control-system" name="gz_ros2_control::GazeboSimROS2ControlPlugin">
+      <parameters>$(find f1_control)/config/ackermann_drive_controller.yaml</parameters>
+      	<ros>
+					<namespace>f1</namespace>
+					<remapping>ackermann_steering_controller/odometry:=odom</remapping>
+          <remapping>ackermann_steering_controller/tf_odometry:=tf</remapping>
+          <parameter name="robot_description">robot_description</parameter>
+				</ros>
     </plugin>
   </gazebo>
@@ -231,5 +248,5 @@
 			<sensor name='lidar' type='gpu_lidar'>
 				<gz_frame_id>lidar_link</gz_frame_id>
-				<topic>scan</topic>
+				<topic>/f1/scan</topic>
 				<update_rate>10</update_rate>
 				<ray>
@@ -257,4 +274,12 @@
 				<visualize>true</visualize>
 			</sensor>
-		</gazebo>
+	</gazebo>
+  <gazebo reference="rear_left_wheel">
+    <mu1>1.2</mu1>
+    <mu2>1.2</mu2>
+  </gazebo>
+  <gazebo reference="rear_right_wheel">
+    <mu1>1.2</mu1>
+    <mu2>1.2</mu2>
+  </gazebo>
 </robot>
